Commit message: Modified files for ridgeback_baxter integration

File: ridgeback_baxter_description/urdf/ridgeback_baxter.urdf.xacro (robot description, xacro)
@@ -1,13 +1,17 @@
-<?xml version="1.0"?>
-<robot name="ridgeback_baxter" xmlns:xacro="http://www.ros.org/wiki/xacro">
-  <xacro:property name="pedestal_height" value="0.565" />
+<?xml version="1.0" ?>
+<robot name="ridgeback_baxter" xmlns:xacro="http://ros.org/wiki/xacro">
+  <xacro:arg name="pedestal" default="true"/>
+  <!--Ridgeback Robot-->
+  <xacro:include filename="$(find ridgeback_description)/urdf/ridgeback.urdf.xacro" />
+  <!-- Baxter Robot -->
+  <xacro:include filename="$(find baxter_description)/urdf/baxter.urdf.xacro" />
+  <xacro:property name="pedestal_height" value="0.85" />
   <xacro:property name="pedestal_diameter" value="0.203" />
   <xacro:property name="pedestal_offset_x" value="0.2" />
-  <xacro:include filename="$(find ridgeback_description)/urdf/ridgeback.urdf.xacro" />
-  <xacro:include filename="$(find baxter_description)/urdf/baxter.urdf" />
+  <!-- Link Baxter and Ridgeback-->
   <joint name="ridgeback_base_to_baxter" type="fixed">
-    <origin rpy="0 0 0" xyz="${pedestal_offset_x} 0 ${pedestal_height}" />
-    <parent link="mid_mount" />
-    <child link="base" />
+      <origin rpy="0 0 0" xyz="${pedestal_offset_x} 0 ${pedestal_height}" />
+      <parent link="chassis_link" />
+      <child link="base" />
   </joint>
 </robot>
